Commit message: Rename rst base naming

File: mhp_robot_ur10_example/ur_description/urdf/ur10.urdf.xacro (robot description, xacro)
@@ -290,5 +290,5 @@
         <origin rpy="0.0 0.0 0.0" xyz="-0.23 -0.33 -0.013"/>
         <geometry>
-          <mesh filename="package://ur_description/meshes/rst_ft/rst_base.stl" scale="0.0255 0.0255 0.0253" />
+          <mesh filename="package://ur_description/meshes/base/base.stl" scale="0.0255 0.0255 0.0253" />
         </geometry>
         <material name="dark_grey">
